Commit message: This is the final commit in the project

File: at_robot_simulation/urdf/driveunit.xacro (robot description, xacro)
@@ -6,4 +6,10 @@
       <mass value="${m}"/>
       <inertia ixx="${m*(3*r*r+h*h)/12}" ixy = "0" ixz = "0" iyy="${m*(3*r*r+h*h)/12}" iyz = "0" izz="${m*r*r/2}"/>
+    </inertial>
+  </xacro:macro>
+  <xacro:macro name="cylinder_y_inertia" params="m r h">
+    <inertial>
+      <mass value="${m}"/>
+      <inertia ixx="${m*(3*r*r+h*h)/12}" ixy = "0" ixz = "0" iyy= "${m*r*r/2}" iyz = "0" izz="${m*(3*r*r+h*h)/12}"/>
     </inertial>
   </xacro:macro>
@@ -31,5 +37,5 @@
     <!--Base plate for the drive unit-->
     <link name="top_plate">
-        <xacro:box_inertia m="1.065" w="0.25" h="0.65" d="0.01" />
+        <xacro:box_inertia m="1.065" w="0.25" h="0.01" d="0.65" />
         <collision name="collision_top_plate">
             <origin rpy="0 1.57 0" xyz="-0.125 0 0"/>
@@ -47,4 +53,7 @@
         </visual>
     </link>
+    <gazebo reference="top_plate">
+            <material>Gazebo/Grey</material>
+    </gazebo>
     <!--Macro for the guide cylinders-->
     <xacro:macro name="guide_cylinders" params="name" >
@@ -67,9 +76,12 @@
             </visual>
         </link>
+        <gazebo reference="${name}">
+            <material>Gazebo/Grey</material>
+        </gazebo>
     </xacro:macro>
     <!--Macro for the middle plates-->
     <xacro:macro name="middle_plates" params="name number origin_rpy origin_xyz" >
         <link name="${name}">
-            <xacro:box_inertia m="0.376" w="0.180" h="0.25" d="0.01" />
+            <xacro:box_inertia m="0.376" w="0.180" h="0.01" d="0.25" />
             <collision name="collision_top_plate">
                 <origin rpy="${origin_rpy}" xyz="${origin_xyz}"/>
@@ -86,9 +98,12 @@
             </visual>
         </link>
+        <gazebo reference="${name}">
+            <material>Gazebo/Grey</material>
+        </gazebo>
     </xacro:macro>
        <!--Macro for the motor-->
     <xacro:macro name="motors" params="name number origin_rpy origin_xyz" >
         <link name="${name}">
-            <xacro:box_inertia m="7.5" w="0.110" h="0.184" d="0.110" />
+            <xacro:box_inertia m="7.5" w="0.110" h="0.110" d="0.184" />
             <collision name="${name}">
                 <origin rpy="${origin_rpy}" xyz="${origin_xyz}"/>
@@ -108,9 +123,12 @@
             </visual>
         </link>
+        <gazebo reference="${name}">
+            <material>Gazebo/Grey</material>
+        </gazebo>
     </xacro:macro>
         <!--Macro for the driveshafts-->
     <xacro:macro name="drive_shafts" params="name" >
         <link name="${name}" >
-            <xacro:cylinder_inertia m="0.2" r="0.015" h="0.05" />
+            <xacro:cylinder_y_inertia m="0.2" r="0.015" h="0.05" />
             <collision name="wheel_${name}">
               <origin rpy="1.57 0 0" xyz="0 0 0"/>
@@ -126,9 +144,12 @@
             </visual>
         </link>
+        <gazebo reference="${name}">
+            <material>Gazebo/Grey</material>
+        </gazebo>
     </xacro:macro>
         <!--Macro for wheels-->
     <xacro:macro name="wheels" params="name origin_rpy number" >
         <link name="${name}" >
-            <xacro:cylinder_inertia m="1.25" r="0.075" h="0.04" />
+            <xacro:cylinder_y_inertia m="1.25" r="0.075" h="0.04" />
             <collision name="guide_cylinders_${name}">
               <origin rpy="1.57 0 0" xyz="0 0 0"/>
@@ -144,4 +165,9 @@
             </visual>
         </link>
+        <gazebo reference="${name}">
+            <material>Gazebo/Orange</material>
+            <mu1>0.8</mu1>
+            <mu2>0.8</mu2>
+        </gazebo>
     </xacro:macro>
     <!--Macro for the hylsor-->
@@ -162,4 +188,7 @@
             </visual>
         </link>
+        <gazebo reference="${name}">
+            <material>Gazebo/Grey</material>
+        </gazebo>
     </xacro:macro>
         <!--Macro for the guide springss-->
@@ -184,4 +213,7 @@
             </visual>
         </link>
+        <gazebo reference="${name}">
+            <material>Gazebo/Blue</material>
+        </gazebo>
     </xacro:macro>
     <!--Macro for the cylinder joints-->
@@ -362,9 +394,9 @@
       <publishWheelJointState>false</publishWheelJointState>
       <wheelAcceleration>false</wheelAcceleration>
-      <wheelTorque>10</wheelTorque>
+      <wheelTorque>20</wheelTorque>
       <publishTf>1</publishTf>
       <odometrySource>world</odometrySource>
     </plugin>
-  </gazebo>
+  </gazebo>-->
   <!--Include the frame and create a joint between them-->
   <xacro:include filename="$(find at_robot_simulation)/urdf/m2wr.xacro" />
@@ -376,5 +408,4 @@
         <limit effort="1000" lower="1000" upper="1000" velocity="0" />
   </joint>
-  <!--Include table and create a joint between them-->
   <xacro:include filename="$(find at_robot_simulation)/urdf/table.xacro" />
   <joint name="frame_to_table" type="fixed">
@@ -389,16 +420,13 @@
     </plugin>
   </gazebo>
-  <!--Include macrodefinitions for the ultrasonic nodes-->
   <xacro:include filename="$(find at_robot_simulation)/urdf/ultrasonic.xacro" />
-  <!--Ultrasonic boxes-->
-  <xacro:ultrasound_boxes name="ultrasound_front_left" theta="0.8" />
-  <xacro:ultrasound_boxes name="ultrasound_front_left_middle" theta="0" />
-  <xacro:ultrasound_boxes name="ultrasound_front_right_middle" theta="0" />
-  <xacro:ultrasound_boxes name="ultrasound_front_right" theta="-0.8" />
-  <xacro:ultrasound_boxes name="ultrasound_back_left" theta="2.3" />
-  <xacro:ultrasound_boxes name="ultrasound_back_left_middle" theta="3.14"/>
-  <xacro:ultrasound_boxes name="ultrasound_back_right_middle" theta="3.14" />
-  <xacro:ultrasound_boxes name="ultrasound_back_right" theta="3.94" />
-  <!--Ultrasonic joints-->
+  <xacro:ultrasound_boxes name="ultrasound_front_left" theta="0.8" topic="front" />
+  <xacro:ultrasound_boxes name="ultrasound_front_left_middle" theta="0" topic="front"/>
+  <xacro:ultrasound_boxes name="ultrasound_front_right_middle" theta="0" topic="front"/>
+  <xacro:ultrasound_boxes name="ultrasound_front_right" theta="-0.8" topic="front"/>
+  <xacro:ultrasound_boxes name="ultrasound_back_left" theta="2.3" topic="back"/>
+  <xacro:ultrasound_boxes name="ultrasound_back_left_middle" theta="3.14" topic="back"/>
+  <xacro:ultrasound_boxes name="ultrasound_back_right_middle" theta="3.14" topic="back"/>
+  <xacro:ultrasound_boxes name="ultrasound_back_right" theta="3.94" topic="back"/>
   <xacro:joint_ultrasonic name="ultrasound_front_left" child="ultrasound_front_left" parent="link_box_front" origin_xyz="0.28 0.65 0.3" />
   <xacro:joint_ultrasonic name="ultrasound_front_left_middle" child="ultrasound_front_left_middle" parent="link_box_front" origin_xyz="0.28 0.45 0.3" />
@@ -408,4 +436,4 @@
   <xacro:joint_ultrasonic name="ultrasound_back_left_middle" child="ultrasound_back_left_middle" parent="link_box_back" origin_xyz="0 0.45 0.3" />
   <xacro:joint_ultrasonic name="ultrasound_back_right_middle" child="ultrasound_back_right_middle" parent="link_box_back" origin_xyz="0 0.25 0.3" />
-  <xacro:joint_ultrasonic name="ultrasound_back_right" child="ultrasound_back_right" parent="link_box_back" origin_xyz="0 0.0 0.3" />-->
+  <xacro:joint_ultrasonic name="ultrasound_back_right" child="ultrasound_back_right" parent="link_box_back" origin_xyz="0 0.0 0.3" />
 </robot>

File: at_robot_simulation/urdf/m2wr.xacro (robot description, xacro)
@@ -14,4 +14,7 @@
               meshscale="1 1 1"
               material="orange"/>
+<gazebo reference="link_chassis">
+  <material>Gazebo/Grey</material>
+</gazebo>
 <xacro:link_collision_box name="link_box_back"
                           rpy="0 0 0"
@@ -127,3 +130,24 @@
                  parent="link_wheel_4"
                  origin_xyz="0.044199 0.00046 -0.054651" />
+<gazebo reference="link_box_back">
+  <material>Gazebo/GreyTransparent</material>
+</gazebo>
+<gazebo reference="link_box_front">
+  <material>Gazebo/GreyTransparent</material>
+</gazebo>
+<gazebo reference="link_box_middle">
+  <material>Gazebo/GreyTransparent</material>
+</gazebo>
+<gazebo reference="link_wheel_1">
+  <material>Gazebo/Orange</material>
+</gazebo>
+<gazebo reference="link_wheel_2">
+  <material>Gazebo/Orange</material>
+</gazebo>
+<gazebo reference="link_wheel_3">
+  <material>Gazebo/Orange</material>
+</gazebo>
+<gazebo reference="link_wheel_4">
+  <material>Gazebo/Orange</material>
+</gazebo>
 </robot>

File: at_robot_simulation/urdf/table.xacro (robot description, xacro)
@@ -13,4 +13,18 @@
     </inertial>
   </xacro:macro>
+  <xacro:macro name="support_legs_inertia" params="m w h d xyz rpy">
+    <inertial>
+      <origin xyz="${xyz}" rpy="${rpy}"/>
+      <mass value="${m}"/>
+      <inertia ixx="${m / 12.0 * (d*d + h*h)}" ixy="0.0" ixz="0.0" iyy="${m / 12.0 * (w*w + h*h)}" iyz="0.0" izz="${m / 12.0 * (w*w + d*d)}"/>
+    </inertial>
+  </xacro:macro>
+  <xacro:macro name="table_inertia" params="m w h d">
+    <inertial>
+      <origin xyz="0 0 0.2" rpy="1.57 0 0"/>
+      <mass value="${m}"/>
+      <inertia ixx="${m / 12.0 * (d*d + h*h)}" ixy="0.0" ixz="0.0" iyy="${m / 12.0 * (w*w + h*h)}" iyz="0.0" izz="${m / 12.0 * (w*w + d*d)}"/>
+    </inertial>
+  </xacro:macro>
     <!--Macro for the side alu profiles-->
     <xacro:macro name="bottom_sides" params="name" >
@@ -34,4 +48,7 @@
             </visual>
         </link>
+        <gazebo reference="${name}">
+            <material>Gazebo/Grey</material>
+        </gazebo>
     </xacro:macro>
     <!--Macro for the bottom front side alu profile-->
@@ -56,9 +73,12 @@
             </visual>
         </link>
+        <gazebo reference="${name}">
+            <material>Gazebo/Grey</material>
+        </gazebo>
     </xacro:macro>
     <!--Macro for the supports to the table-->
-    <xacro:macro name="support_profiles" params="name orgin_rpy origin_xyz" >
-        <link name="${name}" >
-            <xacro:box_inertia m="0.212" w="0.810" h="0.02" d="0.030" />
+    <xacro:macro name="support_profiles" params="name orgin_rpy origin_xyz xyz rpy" >
+        <link name="${name}" >
+            <xacro:support_legs_inertia m="0.212" w="0.810" h="0.02" d="0.030" xyz="${xyz}" rpy="${rpy}"/>
             <collision name="${name}">
               <origin rpy="${orgin_rpy}" xyz="${origin_xyz}"/>
@@ -79,4 +99,7 @@
             </visual>
         </link>
+        <gazebo reference="${name}">
+            <material>Gazebo/Grey</material>
+        </gazebo>
     </xacro:macro>
         <!--Macro for the supports to the table-->
@@ -100,4 +123,7 @@
             </visual>
         </link>
+        <gazebo reference="${name}">
+            <material>Gazebo/Black</material>
+        </gazebo>
     </xacro:macro>
     <!--Macro push link-->
@@ -121,9 +147,12 @@
             </visual>
         </link>
+        <gazebo reference="${name}">
+            <material>Gazebo/Grey</material>
+        </gazebo>
     </xacro:macro>
     <!--Macro table link-->
     <xacro:macro name="table" params="name origin_xyz" >
         <link name="${name}" >
-            <xacro:box_inertia m="1.3" w="0.8" h="0.65" d="0.042" />
+            <xacro:table_inertia m="1.3" w="0.8" h="0.65" d="0.042" />
             <collision name="${name}">
               <origin rpy="-1.57 0 -1.57" xyz="${origin_xyz}"/>
@@ -142,4 +171,7 @@
             </visual>
         </link>
+        <gazebo reference="${name}">
+            <material>Gazebo/Grey</material>
+        </gazebo>
     </xacro:macro>
         <!--Macro wheel link-->
@@ -163,4 +195,7 @@
             </visual>
         </link>
+        <gazebo reference="${name}">
+            <material>Gazebo/Grey</material>
+        </gazebo>
     </xacro:macro>
     <!--Joint to tie the bottom frame together-->
@@ -257,6 +292,6 @@
     <xacro:joint_bottom_table name="right_side" child="right_side" parent="front_alu" origin_xyz="-0.381 -0.304 0" />
     <!--Create table legs-->
-    <xacro:support_profiles name="left_back_leg" orgin_rpy="0 0 0" origin_xyz="0.4 0 0.038"/>
-    <xacro:support_profiles name="right_back_leg" orgin_rpy="0 0 0" origin_xyz="0.4 0 0.038" />
+    <xacro:support_profiles name="left_back_leg" orgin_rpy="0 0 0" origin_xyz="0.4 0 0.038" xyz="0.4 0 0" rpy="0 0 0"/>
+    <xacro:support_profiles name="right_back_leg" orgin_rpy="0 0 0" origin_xyz="0.4 0 0.038" xyz="0.4 0 0" rpy="0 0 0"/>
     <xacro:joint_table_support name="left_back_leg" child="left_back_leg" parent="left_side" origin_xyz="-0.385 -0.03 0.0" orgin_rpy="0 0 0" upper="-0.32" lower="-0.52" />
     <xacro:joint_table_support name="right_back_leg" child="right_back_leg" parent="right_side" origin_xyz="-0.385 0.03 0.0" orgin_rpy="0 0 0" upper="-0.32" lower="-0.52" />
@@ -270,6 +305,6 @@
     <xacro:joint_top_table  name="table_top" child="table_top" parent="push_link" origin_xyz="0 0 0.055" />
     <!--Create legs for top table-->
-    <xacro:support_profiles name="right_front_leg" orgin_rpy="0 0 0" origin_xyz="0.4 0 0.038" />
-    <xacro:support_profiles name="left_front_leg" orgin_rpy="0 0 0" origin_xyz="0.4 0 0.038" />
+    <xacro:support_profiles name="right_front_leg" orgin_rpy="0 0 0" origin_xyz="0.4 0 0.038" xyz="0.4 0 0" rpy="0 0 0"/>
+    <xacro:support_profiles name="left_front_leg" orgin_rpy="0 0 0" origin_xyz="0.4 0 0.038" xyz="0.4 0 0" rpy="0 0 0"/>
     <xacro:joint_table_support name="right_front_leg" child="right_front_leg" parent="table_top" origin_xyz="-0.39 -0.31 0.1" orgin_rpy="0 0 0" upper="0.52" lower="0.32" />
     <xacro:joint_table_support name="left_front_leg" child="left_front_leg" parent="table_top" origin_xyz="-0.39 0.31 0.1" orgin_rpy="0 0 0" upper="0.52" lower="0.32" />

File: at_robot_simulation/urdf/ultrasonic.xacro (robot description, xacro)
@@ -8,5 +8,5 @@
     </xacro:macro>
     <!--Macro for the side alu profiles-->
-    <xacro:macro name="ultrasound_boxes" params="name theta" >
+    <xacro:macro name="ultrasound_boxes" params="name theta topic" >
         <link name="${name}" >
             <xacro:box_inertia m="0.05" w="0.01" h="0.04" d="0.02" />
@@ -58,5 +58,5 @@
                 <alwaysOn>true</alwaysOn>
                 <updateRate>50</updateRate>
-                <topicName>sensor/${name}</topicName>
+                <topicName>sensor/${topic}</topicName>
                 <frameName>${name}</frameName>
                 <radiation>ultrasound</radiation>

Commit message: Added the K-matrix regulator

File: at_robot_simulation/urdf/driveunit.xacro (robot description, xacro)
@@ -132,5 +132,5 @@
             <xacro:cylinder_y_inertia m="0.2" r="0.015" h="0.05" />
             <collision name="wheel_${name}">
-              <origin rpy="1.57 0 0" xyz="0 0 0"/>
+              <origin rpy="1.57 0 0" xyz="0 0 -0.005"/>
               <geometry>
                 <cylinder length="0.05" radius="0.015"/>
@@ -138,5 +138,5 @@
             </collision>
             <visual name="${name}_visual">
-              <origin rpy="1.57 0 0" xyz="0 0 0"/>
+              <origin rpy="1.57 0 0" xyz="0 0 -0.005"/>
               <geometry>
                 <cylinder length="0.05" radius="0.015"/>
@@ -235,4 +235,5 @@
         <axis xyz="0 0 1" />
         <limit effort="1000" lower="-0.03" upper="0" velocity="0.2" />
+        <dynamics damping="0.8" />
       </joint>
     </xacro:macro>
@@ -322,7 +323,19 @@
    <xacro:joint_middle_plates name="left_plate" number="1" child="left_plate" parent="cyl_top_left" origin_xyz="-0.06 -0.05 0"/>
    <xacro:joint_middle_plates name="right_plate" number="1" child="right_plate" parent="cyl_top_right" origin_xyz="-0.06 0.05 0"/>
+   <gazebo reference="left_plate_joint" >
+      <implicitSpringDampner>true</implicitSpringDampner>
+      <springStifness>true</springStifness>
+      <provideFeedback>true</provideFeedback>
+      <springReference>0.0</springReference>
+   </gazebo>
+   <gazebo reference="right_plate_joint" >
+      <implicitSpringDampner>true</implicitSpringDampner>
+      <springStifness>true</springStifness>
+      <provideFeedback>true</provideFeedback>
+      <springReference>0.0</springReference>
+   </gazebo>
    <!--Create motor-->
-   <xacro:motors name ="left_motor" number="1" origin_xyz="-0.02 0.1 0" origin_rpy="0 0 1.57"/>
-   <xacro:motors name ="right_motor" number="2" origin_xyz="0.02 -0.1 0" origin_rpy="0 0 -1.57"/>
+   <xacro:motors name ="left_motor" number="1" origin_xyz="-0.02 0.05 0" origin_rpy="0 0 1.57"/>
+   <xacro:motors name ="right_motor" number="2" origin_xyz="0.02 -0.05 0" origin_rpy="0 0 -1.57"/>
    <xacro:joint_motor_plate name="left_motor" child="left_motor" parent="left_plate" origin_xyz="0 0 -0.055" />
    <xacro:joint_motor_plate name="right_motor" child="right_motor" parent="right_plate" origin_xyz="0 0 -0.055" />
@@ -330,11 +343,11 @@
   <xacro:drive_shafts name="left_shaft" />
   <xacro:drive_shafts name="right_shaft" />
-  <xacro:joint_driveshafts name="left_shaft" child="left_shaft" parent="left_motor" origin_xyz="0 0.117 0" />
-  <xacro:joint_driveshafts name="right_shaft" child="right_shaft" parent="right_motor" origin_xyz="0 -0.117 0" />
+  <xacro:joint_driveshafts name="left_shaft" child="left_shaft" parent="left_motor" origin_xyz="0.01 0.1 0" />
+  <xacro:joint_driveshafts name="right_shaft" child="right_shaft" parent="right_motor" origin_xyz="0.01 -0.1 0" />
   <!--Create wheels-->
   <xacro:wheels name="left_wheel" number="1" origin_rpy="0 0 1.57"/>
   <xacro:wheels name="right_wheel" number="2" origin_rpy="0 0 -1.57"/>
-  <xacro:joint_driveshaft_wheel name="left_wheel" child="left_wheel" parent="left_shaft" origin_xyz="0 0.03 0" />
-  <xacro:joint_driveshaft_wheel name="right_wheel" child="right_wheel" parent="right_shaft" origin_xyz="0 -0.03 0" />
+  <xacro:joint_driveshaft_wheel name="left_wheel" child="left_wheel" parent="left_shaft" origin_xyz="0 0.03 0.0" />
+  <xacro:joint_driveshaft_wheel name="right_wheel" child="right_wheel" parent="right_shaft" origin_xyz="0 -0.03 0.0" />
   <!--Create hylsa for top plate-->
   <xacro:hylsa name="top_left_hylsa" number="1"/>
@@ -384,5 +397,5 @@
       <wheelSeparation>0.65</wheelSeparation>
       <wheelDiameter>0.15</wheelDiameter>
-      <torque>40</torque>
+      <torque>120</torque>
       <commandTopic>cmd_vel</commandTopic>
       <odometryTopic>odom</odometryTopic>
@@ -394,5 +407,5 @@
       <publishWheelJointState>false</publishWheelJointState>
       <wheelAcceleration>false</wheelAcceleration>
-      <wheelTorque>20</wheelTorque>
+      <wheelTorque>60</wheelTorque>
       <publishTf>1</publishTf>
       <odometrySource>world</odometrySource>
